Commit message: Primeiros testes de condução Falta evitar obstáculos

File: p_g3_description/urdf/p_g3.gazebo.xacro (robot description, xacro)
@@ -5,5 +5,4 @@
   <xacro:arg name="imu_visual"    default="false"/>
   <gazebo reference="base_link">
-<!--    <material>Gazebo/Red</material>-->
     <material>Gazebo/${player_color}</material>
   </gazebo>
@@ -144,5 +143,4 @@
           <horizontal_fov>1.085595</horizontal_fov>
           <image>
-<!--              <width>640</width>-->
               <width>900</width>
               <height>480</height>
@@ -178,5 +176,4 @@
           <horizontal_fov>1.085595</horizontal_fov>
           <image>
-<!--              <width>640</width>-->
               <width>900</width>
               <height>480</height>
